File: pt-delay-minima-footswitch.kicad_pcb (KiCad board)
At the start: 2 copper layers, 34 x 24 mm, 10 parts, among them J1 SwitchConn, SW1 SW_Push_3PDT

Commit message: Added versions
Other:
- board text added: "JLCJLCJLCJLC"
- board text added: "v1rev1"
Changed lines of the file:
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@@
       (xy 59 41)
     ) (layer "Edge.Cuts") (width 0.1) (fill none))
+  (gr_text "v1rev1" (at 69.85 46.99) (layer "B.SilkS")
+    (effects (font (size 0.8 0.8) (thickness 0.15)) (justify right mirror))
+  )
+  (gr_text "JLCJLCJLCJLC" (at 69.596 43.18) (layer "B.SilkS")
+    (effects (font (size 0.8 0.8) (thickness 0.15)) (justify mirror))
+  )
   (segment (start 69.881 63.119) (end 72.28 60.72) (width 0.8) (layer "B.Cu") (net 1))
   (segment (start 72.28 60.72) (end 72.28 56.77) (width 0.8) (layer "B.Cu") (net 1))
